File: PDB-SL-OSD.brd (EAGLE design)
At the start: 67.7 x 185.5 mm, 61 parts

Commit message: Update PDB-SL-OSD.brd
Improvements
Connections:
- net S$7 renamed S$42
- new net S$37: AVOUT.1
- new net S$43: AVOUT.2
- net S$1: no longer AVOUT.2
- net S$26: no longer AVOUT.1
Routing:
- net S$26: track 99.5 -> 8.55 mm, vias 1 -> 0
- net S$33: track 0.00 -> 76.5 mm
- net S$43: track 0.00 -> 42.5 mm, vias 0 -> 1
- net S$42: track 71.1 -> 47.8 mm
- net S$7: track 0.00 -> 23.1 mm
- net S$41: track 0.00 -> 20.7 mm
- net S$37: track 0.00 -> 17.0 mm
- net S$1: track 109.3 -> 105.9 mm, vias 2 -> 1
- net S$25: track 94.1 -> 96.9 mm
