File: PDB-SL-OSD.brd (EAGLE design)
At the start: 67.7 x 185.5 mm, 61 parts

Commit message: Update PDB-SL-OSD.brd
Connections:
- removed net S$16: JP5.4
- removed net S$29: JP5.3
- new net S$45: AVIN.2
- new net S$7: JP5.3
- net S$1: now also JP5.4; no longer AVIN.2
Routing:
- net S$45: track 0.00 -> 101.4 mm, vias 0 -> 1
- net S$16: track 79.2 -> 0.00 mm
- net S$29: track 78.8 -> 0.00 mm
- net S$7: track 23.1 -> 76.4 mm
- net S$1: track 105.9 -> 78.2 mm, vias 1 -> 0
- net S$42: track 47.8 -> 71.0 mm
- net S$43: track 42.5 -> 28.6 mm
- net S$26: track 8.55 -> 2.63 mm
- net S$41: track 20.7 -> 17.0 mm
- net S$44: track 0.00 -> 0.72 mm
Other:
- outline, holes or cut-outs redrawn

Commit message: Update PDB-SL-OSD.brd
Parts:
- BUZZER: value F/TMB -> 5V
- C1: value (none) -> 470uF/25V
- L1: value (none) -> 100uH
- LED1, LED10, LED2, LED5, LED6, LED7, LED8, LED9: value (none) -> WHITE
- LED11, LED12, LED13, LED14, LED15, LED16, LED17, LED18, LED19, LED20, LED3, LED4: value (none) -> RED
- R1, R10, R2, R3, R4, R5, R6, R7, R8, R9: value (none) -> 680

Commit message: Update PDB-SL-OSD.brd
Via unconnected Led 1, 2 Fixed
Routing:
- net S$34: track 4.45 -> 0.00 mm, vias 1 -> 0
- net GND: track 10.9 -> 15.4 mm, vias 1 -> 2
Changed lines of the file:
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@@
 <wire x1="37.465" y1="115.189" x2="37.465" y2="115.57" width="0.4064" layer="1"/>
-</signal>
-<signal name="S$34">
-<via x="54.9275" y="173.355" extent="1-16" drill="0.6"/>
-<wire x1="54.9275" y1="173.355" x2="59.3725" y2="173.355" width="0.3048" layer="1"/>
 </signal>
 <signal name="S$13">
@@
 <wire x1="17.18" y1="13.46" x2="17.24" y2="13.52" width="0.4064" layer="16"/>
 <wire x1="17.24" y1="13.52" x2="18.66" y2="13.52" width="0.4064" layer="16"/>
+<via x="54.9275" y="173.355" extent="1-16" drill="0.6"/>
+<wire x1="54.9275" y1="173.355" x2="59.3725" y2="173.355" width="0.3048" layer="1"/>
 <wire x1="59.944" y1="161.2265" x2="57.912" y2="160.782" width="0" layer="19" extent="1-1"/>
 <wire x1="29.845" y1="115.189" x2="29.337" y2="117.0305" width="0" layer="19" extent="1-1"/>
@@
 </signal>
 </signals>
+<errors>
+</errors>
 </board>
 </drawing>
